Commit message: complete autonomous

File: src/my_robot_description/urdf/my_robot.urdf (robot description, URDF)
Before this commit: robot my_robot, 7 links, 6 joints
Links:
- link base_link: mass 1.0 -> 1.5
- link base_scan: mass 0.05 -> 0.5
- link camera_link: mass 0.02 -> 0.3
Joints:
- joint caster_joint: axis (none) -> 0 1 0; type fixed -> continuous
